File: Hardware/uC_TP_Boussole_mb/Current_NCS199A3RSQT2G.kicad_sch (KiCad schematic)
At the start: 0 parts

Commit message: starting pin out nucleo
Parts:
- added R601: R_Small, Resistor_SMD:R_0402_1005Metric, symbol Device:R_Small
- added U601: ~, symbol NCS199A3RSQT2G:NCS199A3RSQT2G
Connections:
- new net +3.3V: U601.3 (Vs)
- new net GND: U601.1 (REF), U601.2 (GND)
- new net Imes: U601.6 (OUT)
- new net Load: R601.2, U601.5 (IN-)
- new net Supply: R601.1, U601.4 (IN+)

Commit message: update ppcb
Parts:
- added C601: 100n, Capacitor_SMD:C_0402_1005Metric, symbol Device:C_Small
- R601: value R_Small -> 30m
- U601: footprint (none) -> Package_TO_SOT_SMD:SOT-363_SC-70-6; MPN (none) -> NCS199A3RSQT2G
Connections:
- net +3.3V: now also C601.1
- net GND: now also C601.2
Other:
- note added: "Max Current 500mA Min Current 0mA Vref = 0V Vout = 3V @ Imes = 0.5A Rsense = 30mohm"
Changed lines of the file:
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@@
+	(wire
+		(pts
+			(xy 189.23 86.36) (xy 189.23 88.9)
+		)
+		(stroke
+			(width 0)
+			(type default)
+		)
+	)
 	(wire
 		(pts
@@
 	(wire
 		(pts
+			(xy 189.23 80.01) (xy 189.23 81.28)
+		)
+		(stroke
+			(width 0)
+			(type default)
+		)
+	)
+	(wire
+		(pts
 			(xy 113.03 78.74) (xy 127 78.74)
 		)
@@
 			(width 0)
 			(type default)
+		)
+	)
+	(text "Max Current 500mA\nMin Current 0mA\nVref = 0V\nVout = 3V @ Imes = 0.5A\nRsense = 30mohm"
+		(exclude_from_sim no)
+		(at 120.65 107.95 0)
+		(effects
+			(font
+				(size 1.27 1.27)
+			)
+			(justify left top)
 		)
 	)
@@
 			)
 		)
-		(property "Footprint" ""
+		(property "Footprint" "Package_TO_SOT_SMD:SOT-363_SC-70-6"
 			(at 139.7 85.09 0)
 			(effects
@@
 			)
 		)
-		(property "Datasheet" ""
+		(property "Datasheet" "https://www.mouser.fr/datasheet/2/308/1/NCS199A1R_D-2317315.pdf"
 			(at 139.7 85.09 0)
 			(effects
@@
 		)
 		(property "Description" ""
+			(at 139.7 85.09 0)
+			(effects
+				(font
+					(size 1.27 1.27)
+				)
+				(hide yes)
+			)
+		)
+		(property "MPN" "NCS199A3RSQT2G"
 			(at 139.7 85.09 0)
 			(effects
@@
 	)
 	(symbol
+		(lib_id "Device:C_Small")
+		(at 189.23 83.82 0)
+		(unit 1)
+		(exclude_from_sim no)
+		(in_bom yes)
+		(on_board yes)
+		(dnp no)
+		(fields_autoplaced yes)
+		(property "Reference" "C601"
+			(at 191.77 82.5562 0)
+			(effects
+				(font
+					(size 1.27 1.27)
+				)
+				(justify left)
+			)
+		)
+		(property "Value" "100n"
+			(at 191.77 85.0962 0)
+			(effects
+				(font
+					(size 1.27 1.27)
+				)
+				(justify left)
+			)
+		)
+		(property "Footprint" "Capacitor_SMD:C_0402_1005Metric"
+			(at 189.23 83.82 0)
+			(effects
+				(font
+					(size 1.27 1.27)
+				)
+				(hide yes)
+			)
+		)
+		(property "Datasheet" "~"
+			(at 189.23 83.82 0)
+			(effects
+				(font
+					(size 1.27 1.27)
+				)
+				(hide yes)
+			)
+		)
+		(property "Description" "Unpolarized capacitor, small symbol"
+			(at 189.23 83.82 0)
+			(effects
+				(font
+					(size 1.27 1.27)
+				)
+				(hide yes)
+			)
+		)
+		(pin "1"
+		)
+		(pin "2"
+		)
+		(instances
+			(project "uC_TP_Boussole_mb"
+				(path "/2e9feef3-d2ce-488a-99fa-e1de5099ffc3/864c7139-0ed0-4610-9ca7-6ef011edb53c"
+					(reference "C601")
+					(unit 1)
+				)
+			)
+		)
+	)
+	(symbol
 		(lib_id "power:GND")
 		(at 139.7 93.98 0)
@@
 	)
 	(symbol
+		(lib_id "power:GND")
+		(at 189.23 88.9 0)
+		(unit 1)
+		(exclude_from_sim no)
+		(in_bom yes)
+		(on_board yes)
+		(dnp no)
+		(fields_autoplaced yes)
+		(property "Reference" "#PWR0605"
+			(at 189.23 95.25 0)
+			(effects
+				(font
+					(size 1.27 1.27)
+				)
+				(hide yes)
+			)
+		)
+		(property "Value" "GND"
+			(at 189.23 93.98 0)
+			(effects
+				(font
+					(size 1.27 1.27)
+				)
+			)
+		)
+		(property "Footprint" ""
+			(at 189.23 88.9 0)
+			(effects
+				(font
+					(size 1.27 1.27)
+				)
+				(hide yes)
+			)
+		)
+		(property "Datasheet" ""
+			(at 189.23 88.9 0)
+			(effects
+				(font
+					(size 1.27 1.27)
+				)
+				(hide yes)
+			)
+		)
+		(property "Description" "Power symbol creates a global label with name \"GND\" , ground"
+			(at 189.23 88.9 0)
+			(effects
+				(font
+					(size 1.27 1.27)
+				)
+				(hide yes)
+			)
+		)
+		(pin "1"
+		)
+		(instances
+			(project "uC_TP_Boussole_mb"
+				(path "/2e9feef3-d2ce-488a-99fa-e1de5099ffc3/864c7139-0ed0-4610-9ca7-6ef011edb53c"
+					(reference "#PWR0605")
+					(unit 1)
+				)
+			)
+		)
+	)
+	(symbol
+		(lib_id "power:+3.3V")
+		(at 189.23 80.01 0)
+		(unit 1)
+		(exclude_from_sim no)
+		(in_bom yes)
+		(on_board yes)
+		(dnp no)
+		(fields_autoplaced yes)
+		(property "Reference" "#PWR0604"
+			(at 189.23 83.82 0)
+			(effects
+				(font
+					(size 1.27 1.27)
+				)
+				(hide yes)
+			)
+		)
+		(property "Value" "+3.3V"
+			(at 189.23 74.93 0)
+			(effects
+				(font
+					(size 1.27 1.27)
+				)
+			)
+		)
+		(property "Footprint" ""
+			(at 189.23 80.01 0)
+			(effects
+				(font
+					(size 1.27 1.27)
+				)
+				(hide yes)
+			)
+		)
+		(property "Datasheet" ""
+			(at 189.23 80.01 0)
+			(effects
+				(font
+					(size 1.27 1.27)
+				)
+				(hide yes)
+			)
+		)
+		(property "Description" "Power symbol creates a global label with name \"+3.3V\""
+			(at 189.23 80.01 0)
+			(effects
+				(font
+					(size 1.27 1.27)
+				)
+				(hide yes)
+			)
+		)
+		(pin "1"
+		)
+		(instances
+			(project "uC_TP_Boussole_mb"
+				(path "/2e9feef3-d2ce-488a-99fa-e1de5099ffc3/864c7139-0ed0-4610-9ca7-6ef011edb53c"
+					(reference "#PWR0604")
+					(unit 1)
+				)
+			)
+		)
+	)
+	(symbol
 		(lib_id "power:+3.3V")
 		(at 139.7 76.2 0)
@@
 			)
 		)
-		(property "Value" "R_Small"
+		(property "Value" "30m"
 			(at 115.57 83.8199 0)
 			(effects

Commit message: ddd
Parts:
- U601: value ~ -> NCS199A3RSQT2G
Changed lines of the file:
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@@
 		(on_board yes)
 		(dnp no)
-		(fields_autoplaced yes)
 		(property "Reference" "U601"
 			(at 163.83 82.712 0)
@@
 			)
 		)
-		(property "Value" "~"
-			(at 163.83 84.6171 0)
+		(property "Value" "NCS199A3RSQT2G"
+			(at 149.86 75.692 0)
 			(effects
 				(font

Commit message: bom
Parts:
- R601: MPN (none) -> ERJ2RKF30R1X
Changed lines of the file:
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@@
+			)
+		)
+		(property "MPN" "ERJ2RKF30R1X"
+			(at 113.03 82.55 0)
+			(effects
+				(font
+					(size 1.27 1.27)
+				)
+				(hide yes)
 			)
 		)
